Commit message: Add parent and origin params to position sensors and root joint

File: micro_epsilon_scancontrol_description/urdf/scancontrol_26x0_29x0_25_macro.xacro (robot description, xacro)
@@ -2,5 +2,5 @@
 <robot xmlns:xacro="http://wiki.ros.org/xacro">
   <!-- Macro for both 26x0 and 29x0 - 25 scan control sensor productlines -->
-  <xacro:macro name="microepsilon_scancontrol_26x0_29x0_25" params="prefix">
+  <xacro:macro name="sensor_2610_100" params="parent *origin prefix">
     <link name="${prefix}base_link">
       <visual>
@@ -21,4 +21,9 @@
     </link>
     <link name="${prefix}aperture_frame" />
+    <joint name="${prefix}_joint" type="fixed">
+      <xacro:insert_block name="origin" />
+      <parent link="${parent}" />
+      <child link="${prefix}base_link" />
+    </joint>
     <joint name="${prefix}base_link-${prefix}aperture_frame" type="fixed">
       <origin xyz="0 0 0" rpy="${pi} 0 ${pi/2}" />
